Commit message: Model and thruster frames

File: mercury_descriptions/common/xacro/snippets.xacro (robot description, xacro)
@@ -12,9 +12,9 @@
         </joint>
         <link name="${namespace}/thruster_${thruster_id}">
-            <!-- <visual>
+            <visual>
                 <geometry>
-                    <mesh filename="${mesh_filename}" scale="1 1 1" />
+                    <mesh filename="package://riptide_descriptions2/meshes/Propeller.dae" scale="1 1 1" />
                 </geometry>
-            </visual> -->
+            </visual>
         </link>
     </xacro:macro>

File: mercury_descriptions/mercury/xacro/mercury_base.xacro (robot description, xacro)
@@ -12,4 +12,10 @@
             <transparency>0.8</transparency>
         </visual> -->
+            <visual>
+                <geometry>
+                    <mesh filename="package://mercury_meshes/meshes/mercury/model.dae" scale="1 1 1"/>
+                </geometry>
+                <transparency>0.8</transparency>
+            </visual>
         </link>
         <!-- <xacro:include filename="$(find mercury_descriptions)/mercury/robot_sensors.xacro" /> -->

Commit message: Depth sensor frame and raw msg

File: mercury_descriptions/common/xacro/snippets.xacro (robot description, xacro)
@@ -47,3 +47,16 @@
         </xacro:if>
     </xacro:macro>
+    <!-- Depth Sensor-->
+    <xacro:macro name="depth_macro" params="namespace parent_link config">
+        <xacro:if value="${'depth' in config}">
+            <link name="${namespace}/depth_link" />
+            <xacro:property name="depth" value="${config['depth']}"/>
+            <joint name="${namespace}/depth_joint" type="fixed">
+                <origin xyz="${depth['pose'][0]} ${depth['pose'][1]} ${depth['pose'][2]}"
+                        rpy="${depth['pose'][3]} ${depth['pose'][4]} ${depth['pose'][5]}" />
+                <parent link="${parent_link}" />
+                <child link="${namespace}/depth_link" />
+            </joint>
+        </xacro:if>
+    </xacro:macro>
 </robot>

File: mercury_descriptions/mercury/xacro/mercury_base.xacro (robot description, xacro)
@@ -21,4 +21,8 @@
         <!-- <xacro:include filename="$(find mercury_descriptions)/mercury/robot_sensors.xacro" /> -->
         <!-- <xacro:include filename="$(find riptide_descriptions2)/urdf/robot_actuators.xacro" /> -->
+        <xacro:all_thrusters_macro
+            namespace="${namespace}"
+            thrusters="${config['thrusters']}"
+            index="0" />
         <xacro:imu_macro
             namespace="${namespace}"
@@ -26,8 +30,8 @@
             parent_link="${namespace}/base_link"
             config="${config}" />
-        <xacro:all_thrusters_macro
+        <xacro:depth_macro
             namespace="${namespace}"
-            thrusters="${config['thrusters']}"
-            index="0" />
+            parent_link="${namespace}/base_link"
+            config="${config}" />
   </xacro:macro>
 </robot>

Commit message: Updated xacro for zed, moved zed/imu frames in config

File: mercury_descriptions/common/xacro/snippets.xacro (robot description, xacro)
@@ -60,3 +60,27 @@
         </xacro:if>
     </xacro:macro>
+    <!-- Cameras -->
+    <xacro:macro name="cameras_macro" params="namespace parent_link cameras">
+        <xacro:if value="${cameras != []}">
+            <xacro:property name="camera" value="${cameras[0]}"/>
+            <xacro:property name="camera_base_link" value="${namespace}/${camera['name']}_base_link"/>
+            <link name="${camera_base_link}" />
+            <joint name="${camera_base_link}_joint" type="fixed">
+                <parent link="${parent_link}"/>
+                <child link="${camera_base_link}"/>
+                <origin xyz="${camera['pose'][0]} ${camera['pose'][1]} ${camera['pose'][2]}"
+                        rpy="${camera['pose'][3]} ${camera['pose'][4]} ${camera['pose'][5]}"/>
+            </joint>
+            <!-- Stereo Camera(s) -->
+            <xacro:if value="${camera['type'] == 'stereo'}">
+                <xacro:stereo_macro
+                    namespace="${namespace}"
+                    parent_link="${namespace}/${camera['name']}_base_link"
+                    name="${camera['name']}"
+                    baseline="${camera['baseline']}">
+                    <origin xyz="0 ${camera['baseline'] / 2} 0" />
+                </xacro:stereo_macro>
+            </xacro:if>
+        </xacro:if>
+    </xacro:macro>
 </robot>

File: mercury_descriptions/mercury/xacro/mercury.xacro (robot description, xacro)
@@ -15,6 +15,3 @@
         namespace="$(arg namespace)"
         config="${config}" />
-    <xacro:if value="$(arg use_zed_camera)">
-        <xacro:include filename="$(arg zed_xacro_path)" />
-    </xacro:if>
 </robot>

File: mercury_descriptions/mercury/xacro/mercury_base.xacro (robot description, xacro)
@@ -34,4 +34,8 @@
             parent_link="${namespace}/base_link"
             config="${config}" />
+        <xacro:cameras_macro
+            namespace="${namespace}"
+            parent_link="${namespace}/base_link"
+            cameras="${config['cameras']}" />
   </xacro:macro>
 </robot>
