Commit message: added dvl to xacro for sim

File: mercury_descriptions/mercury/xacro/mercury_base.xacro (robot description, xacro)
@@ -19,4 +19,11 @@
             </visual>
         </link>
+        <link name="${namespace}/dvl_link">
+        </link>
+        <joint name="dvl_joint" type="fixed">
+            <parent link="${namespace}/base_link"/>
+            <child link="${namespace}/dvl_link"/>
+            <origin xyz="0.0 0 0.0" rpy="0 0 0"/>
+        </joint>
         <!-- <xacro:include filename="$(find mercury_descriptions)/mercury/robot_sensors.xacro" /> -->
         <!-- <xacro:include filename="$(find riptide_descriptions2)/urdf/robot_actuators.xacro" /> -->

Commit message: Base center frame for EKF

File: mercury_descriptions/mercury/xacro/mercury_base.xacro (robot description, xacro)
@@ -5,4 +5,10 @@
     <xacro:macro name="robot_base"
         params="namespace config">
+        <link name="${namespace}/base_center"/>
+            <joint name="${namespace}/base_center_to_base_link" type="fixed">
+                <parent link="${namespace}/base_center"/>
+                <child link="${namespace}/base_link"/>
+                <origin xyz="${config['robot_center'][0]} ${config['robot_center'][1]} ${config['robot_center'][2]}" rpy="0 0 0"/>
+            </joint>
         <link name="${namespace}/base_link">
         <!-- <visual>
