Commit message: mercury_sim xacro to have the fake dvl

File: mercury_descriptions/mercury/xacro/mercury.xacro (robot description, xacro)
@@ -4,4 +4,5 @@
     <xacro:arg name="use_zed_camera" default="false" />
     <xacro:arg name="zed_xacro_path" default="" />
+    <xacro:arg name="sim_enabled" default="false" />
     <!-- Include the Robot macro file -->
     <xacro:include filename="$(find mercury_descriptions)/mercury/xacro/mercury_base.xacro" />
@@ -15,3 +16,8 @@
         namespace="$(arg namespace)"
         config="${config}" />
+    <xacro:if value="$(arg sim_enabled)">
+        <xacro:include filename="$(find mercury_descriptions)/mercury/xacro/mercury_sim.xacro" />
+        <xacro:sim_setup
+            namespace="$(arg namespace)" />
+    </xacro:if>
 </robot>

File: mercury_descriptions/mercury/xacro/mercury_base.xacro (robot description, xacro)
@@ -19,11 +19,4 @@
             </visual>
         </link>
-        <link name="${namespace}/dvl_link">
-        </link>
-        <joint name="dvl_joint" type="fixed">
-            <parent link="${namespace}/base_link"/>
-            <child link="${namespace}/dvl_link"/>
-            <origin xyz="0.0 0 0.0" rpy="0 0 0"/>
-        </joint>
         <!-- <xacro:include filename="$(find mercury_descriptions)/mercury/robot_sensors.xacro" /> -->
         <!-- <xacro:include filename="$(find riptide_descriptions2)/urdf/robot_actuators.xacro" /> -->
